File: modules/line_out/line_out.kicad_pcb (KiCad board)
At the start: 2 copper layers, 30.5 x 68.6 mm, 4 parts

Commit message: Finalized the line_out module.
Parts:
- added C1: 0.1uf, Capacitor_SMD:C_0402_1005Metric, F.Cu at (56.5, 85.6)
- added C2: 2.2uf, Capacitor_SMD:C_0603_1608Metric, F.Cu at (73.8, 86.4)
- added C3: 2.2uf, Capacitor_SMD:C_0603_1608Metric, F.Cu at (50.8, 86.4)
- added C4: 100pf, Capacitor_SMD:C_0402_1005Metric, F.Cu at (53.3, 83.0)
- added C5: 100pf, Capacitor_SMD:C_0402_1005Metric, F.Cu at (70.6, 83.0)
- added OUT: AudioJack3, BreadModular_AudioJacks:Jack_3.5mm_QingPu_WQP-PJ366ST_Vertical, F.Cu at (62.0, 67.9)
- added R1: 1k, Resistor_SMD:R_0402_1005Metric, F.Cu at (59.4, 54.6)
- added R2: 1k, Resistor_SMD:R_0402_1005Metric, F.Cu at (62.6, 54.6)
- added R3: 100k, Resistor_SMD:R_0402_1005Metric, F.Cu at (67.9, 85.6)
- added R4: 100k, Resistor_SMD:R_0402_1005Metric, F.Cu at (53.3, 85.6)
- added R5: 33k, Resistor_SMD:R_0402_1005Metric, F.Cu at (56.5, 83.1)
- added R7: 1k, Resistor_SMD:R_0402_1005Metric, F.Cu at (50.7, 83.4)
- added R8: 33k, Resistor_SMD:R_0402_1005Metric, F.Cu at (67.9, 83.1)
- added R9: 1k, Resistor_SMD:R_0402_1005Metric, F.Cu at (73.8, 83.2)
- added U1: TL072, Package_SO:SOIC-8-1EP_3.9x4.9mm_P1.27mm_EP2.29x3mm, F.Cu at (62.2, 84.5)
- renumbered INPUT1 to INPUT, OUTPUT2 to OUTPUT
Connections:
- INPUT pad 1: unconnected-(INPUT1-Pin_1-Pad1) -> IN_L
- INPUT pad 2: unconnected-(INPUT1-Pin_2-Pad2) -> IN_R
- INPUT pad 3: unconnected-(INPUT1-Pin_3-Pad3) -> Net-(INPUT1-Pin_3)
- INPUT pad 4: unconnected-(INPUT1-Pin_4-Pad4) -> Net-(INPUT1-Pin_3)
- INPUT pad 5: unconnected-(INPUT1-Pin_5-Pad5) -> Net-(INPUT1-Pin_3)
- OUTPUT pad 1: unconnected-(OUTPUT2-Pin_1-Pad1) -> OUT_L
- OUTPUT pad 2: unconnected-(OUTPUT2-Pin_2-Pad2) -> OUT_R
- OUTPUT pad 3: unconnected-(OUTPUT2-Pin_3-Pad3) -> Net-(OUTPUT2-Pin_3)
- OUTPUT pad 4: unconnected-(OUTPUT2-Pin_4-Pad4) -> Net-(OUTPUT2-Pin_3)
- OUTPUT pad 5: unconnected-(OUTPUT2-Pin_5-Pad5) -> Net-(OUTPUT2-Pin_3)
Routing:
- net GND: track 10.2 -> 121.9 mm, vias 0 -> 2
- net +2.5V: track 0.00 -> 62.4 mm, vias 0 -> 2
- net IN_R: track 0.00 -> 60.9 mm
- net OUT_R: track 0.00 -> 57.3 mm, vias 0 -> 2
- net OUT_L: track 0.00 -> 55.4 mm, vias 0 -> 2
- net IN_L: track 0.00 -> 47.2 mm
- net +5V: track 10.2 -> 51.3 mm, vias 0 -> 1
- net Net-(C3-Pad1): track 0.00 -> 14.1 mm
- net Net-(C2-Pad1): track 0.00 -> 11.4 mm
- net Net-(U1A--): track 0.00 -> 8.12 mm
- net Net-(U1B--): track 0.00 -> 8.11 mm
- net Net-(OUTPUT2-Pin_3): track 0.00 -> 5.08 mm
- net Net-(INPUT1-Pin_3): track 0.00 -> 5.08 mm
- net Net-(C2-Pad2): track 0.00 -> 3.29 mm
- net Net-(C3-Pad2): track 0.00 -> 3.14 mm
Other:
- board text added: "L"
- board text added: "MULT"
- board text added: "R"
