File: modules/line_out/line_out.kicad_sch (KiCad schematic)
At the start: 21 parts, among them J1 AudioJack3, U1 TL072

Commit message: Finalized the line_out module.
Parts:
- added C4, C5: 100pf, Capacitor_SMD:C_0402_1005Metric, symbol Device:C
- added V3: VSIN, symbol Simulation_SPICE:VSIN
Connections:
- net GND: now also V3.2
- net IN_R: now also V3.1
- net at C2.1, R8.1, U1.7: now also C5.1
- net at C3.1, R5.1, U1.1: now also C4.1
- net at R4.1, R5.2, U1.2 (-): now also C4.2
- net at R3.1, R8.2, U1.6 (-): now also C5.2
Other:
- moved on the sheet: C2, R10, R3, R8, R9, U1B
