File: modules/4_mix/4_mix.kicad_pcb (KiCad board)
At the start: 2 copper layers, 61 x 68.6 mm, 38 parts, among them U1 TL072, U2 TL072, U3 TL072

Commit message: Add missing production files for 4_mix
Parts:
- U1, U2, U3: value TL072 -> MCP6002
Changed lines of the file:
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@@
 			)
 		)
-		(property "Value" "TL072"
+		(property "Value" "MCP6002"
 			(at 0 3.4 0)
 			(layer "F.Fab")
@@
 			)
 		)
-		(property "Value" "TL072"
+		(property "Value" "MCP6002"
 			(at 0 3.4 0)
 			(layer "F.Fab")
@@
 			)
 		)
-		(property "Value" "TL072"
+		(property "Value" "MCP6002"
 			(at 0 3.4 0)
 			(layer "F.Fab")
