File: modules/jvca/jvca.kicad_pcb (KiCad board)
At the start: 2 copper layers, 30.5 x 68.6 mm, 4 parts

Commit message: Implemented JVCA PCB
Parts:
- removed OUTPUT2: Conn_01x05_Socket, Connector_PinSocket_2.54mm:PinSocket_1x05_P2.54mm_Vertical
- added C1: 0.1uf, Capacitor_SMD:C_0402_1005Metric, F.Cu at (49.7, 87.5)
- added C2: 4.7uf, Capacitor_SMD:C_1206_3216Metric, F.Cu at (74.9, 88.5)
- added C3: 0.1uf, Capacitor_SMD:C_0402_1005Metric, F.Cu at (71.7, 93.9)
- added C4: 0.1uf, Capacitor_SMD:C_0402_1005Metric, F.Cu at (57.8, 93.9)
- added CV BIAS: 1k, BreadModular_Pots:Potentiometer_RV09, F.Cu at (59.9, 81.7)
- added CV GAIN: 1M, BreadModular_Pots:Potentiometer_RV09, F.Cu at (59.6, 65.0)
- added OUTPUT: Conn_01x05_Socket, Connector_PinSocket_2.54mm:PinSocket_1x05_P2.54mm_Vertical, F.Cu at (73.7, 45.7)
- added Q1: 2N5457, Package_TO_SOT_THT:TO-92L_Wide, F.Cu at (71.1, 100.8)
- added R1: 200k, Resistor_SMD:R_0402_1005Metric, F.Cu at (63.0, 91.6)
- added R10: 100k, Resistor_SMD:R_0402_1005Metric, F.Cu at (75.1, 93.1)
- added R11: 1M, Resistor_SMD:R_0402_1005Metric, F.Cu at (68.7, 102.2)
- added R12: 200k, Resistor_SMD:R_0402_1005Metric, F.Cu at (61.0, 91.6)
- added R13: 1k, Resistor_SMD:R_0402_1005Metric, F.Cu at (49.5, 82.5)
- added R14: 1k, Resistor_SMD:R_0402_1005Metric, F.Cu at (61.0, 89.4)
- added R15: 1k, Resistor_SMD:R_0402_1005Metric, F.Cu at (59.2, 101.0)
- added R16: 1k, Resistor_SMD:R_0402_1005Metric, F.Cu at (63.4, 101.0)
- added R2: 22k, Resistor_SMD:R_0402_1005Metric, F.Cu at (63.0, 90.2)
- added R3: 51k, Resistor_SMD:R_0402_1005Metric, F.Cu at (75.1, 82.3)
- added R4: 100k, Resistor_SMD:R_0402_1005Metric, F.Cu at (49.7, 93.3)
- added R5: 51k, Resistor_SMD:R_0402_1005Metric, F.Cu at (75.1, 84.9)
- added R6: 22k, Resistor_SMD:R_0402_1005Metric, F.Cu at (49.7, 89.8)
- added R7: 100k, Resistor_SMD:R_0402_1005Metric, F.Cu at (63.0, 87.9)
- added R8: 2k, Resistor_SMD:R_0402_1005Metric, F.Cu at (71.9, 82.3)
- added R9: 1M, Resistor_SMD:R_0402_1005Metric, F.Cu at (75.1, 95.9)
- added U1: MCP6002-xSN, Package_SO:SOIC-8-1EP_3.9x4.9mm_P1.27mm_EP2.29x3mm, F.Cu at (55.2, 90.2)
- added U2: MCP6002-xSN, Package_SO:SOIC-8-1EP_3.9x4.9mm_P1.27mm_EP2.29x3mm, F.Cu at (68.6, 90.0)
- renumbered INPUT1 to INPUT
Connections:
- INPUT pad 1: unconnected-(INPUT1-Pin_1-Pad1) -> V_IN
- INPUT pad 2: unconnected-(INPUT1-Pin_2-Pad2) -> CV
- INPUT pad 3: unconnected-(INPUT1-Pin_3-Pad3) -> Net-(INPUT1-Pin_3)
- INPUT pad 4: unconnected-(INPUT1-Pin_4-Pad4) -> Net-(INPUT1-Pin_3)
- INPUT pad 5: unconnected-(INPUT1-Pin_5-Pad5) -> Net-(INPUT1-Pin_3)
Routing:
- net +5V: track 10.2 -> 134.6 mm, vias 0 -> 4
- net +2.5V: track 0.00 -> 69.9 mm, vias 0 -> 5
- net GND: track 10.2 -> 78.9 mm, vias 0 -> 4
- net V_IN: track 0.00 -> 61.9 mm, vias 0 -> 2
- net JFET_OUT: track 0.00 -> 57.9 mm, vias 0 -> 2
- net V_OUT: track 0.00 -> 57.7 mm, vias 0 -> 4
- net Net-(R3-Pad2): track 0.00 -> 30.2 mm
- net CV: track 0.00 -> 28.4 mm
- net Net-(U1B--): track 0.00 -> 25.2 mm
- net Net-(R10-Pad1): track 0.00 -> 22.9 mm, vias 0 -> 2
- net Net-(Q1-G): track 0.00 -> 14.4 mm
- net Net-(U2B--): track 0.00 -> 13.3 mm
- net Net-(R13-Pad2): track 0.00 -> 12.5 mm
- net Net-(R8-Pad1): track 0.00 -> 8.45 mm
- net Net-(C2-Pad1): track 0.00 -> 7.10 mm
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Other:
- board text added: "1V"
- board text added: "3V"
- board text added: "AUDIO"
- board text added: "CV"
- board text added: "JVCA 0.1.0"
- board text added: "MULT"
- board text removed: "JVCA 0.0.0"
