File: modules/ar_env/ar_env.kicad_sch (KiCad schematic)
At the start: 25 parts, among them U1 MCP6002-xSN, U2 MCP6002-xSN

Commit message: Finalize the PCB
Parts:
- removed R1, R2: 1k, Resistor_SMD:R_0402_1005Metric, symbol Device:R
- C1, C3: footprint Capacitor_SMD:C_1206_3216Metric -> Capacitor_SMD:C_0402_1005Metric
- D1, D2, D3: footprint Diode_SMD:D_SOD-323 -> Diode_SMD:D_SOD-323_HandSoldering

Commit message: Changed the 6.8k resistor package. Used 0603 package due to availability in JLCPCB
Parts:
- R5: footprint Resistor_SMD:R_0402_1005Metric -> Resistor_SMD:R_0603_1608Metric
Changed lines of the file:
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@@
 			)
 		)
-		(property "Footprint" "Resistor_SMD:R_0402_1005Metric"
+		(property "Footprint" "Resistor_SMD:R_0603_1608Metric"
 			(at 52.07 80.518 90)
 			(effects
