File: modules/wave/wave.kicad_sch (KiCad schematic)
At the start: 30 parts, among them U1 MCP6002-xSN, U2 MCP6002-xSN

Commit message: Finish schematics
Parts:
- added C9: 22uf, Capacitor_SMD:C_0805_2012Metric, symbol Device:C
- added INPUT2: Caps, Connector_PinSocket_2.54mm:PinSocket_1x05_P2.54mm_Vertical, symbol Connector:Conn_01x05_Socket
- INPUT1: value Conn_01x05_Socket -> Cap Connect
- OUTPUT2: value Conn_01x05_Socket -> Output Waves
Connections:
- net CAP_HIGH: now also INPUT2.3 (Pin_3); no longer R5.1, U2.2 (-), U2.5 (+)
- net CAP_LFO: now also INPUT2.1 (Pin_1)
- net CAP_LOW: now also INPUT2.2 (Pin_2)
- net GND: now also C9.2
- net OUT_SINE: now also OUTPUT2.5 (Pin_5)
- net OUT_SQUARE: now also OUTPUT2.1 (Pin_1), OUTPUT2.2 (Pin_2)
- net OUT_TRI: now also OUTPUT2.3 (Pin_3), OUTPUT2.4 (Pin_4)
- net CAP_CONNECT: now reaches INPUT1.1 (Pin_1)
- net CAP_CONNECT: now also INPUT1.2 (Pin_2), INPUT1.3 (Pin_3), INPUT1.4 (Pin_4), INPUT1.5 (Pin_5), R5.1, U2.2 (-), U2.5 (+)
- new net CAP_CUSTOM: C9.1, INPUT2.4 (Pin_4), INPUT2.5 (Pin_5)
Other:
- note added: "Connect CAP_CONNECT with CAP_XXX ------------------------ Otherwise, simulations won't work."
- moved on the sheet: INPUT1, R1, R2, U1C, U2C, V1

Commit message: Initiate the PCB layut
Parts:
- added C10, C11: 0.1uf, Capacitor_SMD:C_0402_1005Metric, symbol Device:C
- C1, C2, C3, C4, C5, C6, C7, C8: footprint (none) -> Capacitor_SMD:C_0402_1005Metric
- R1, R10, R11, R13, R2, R3, R4, R5, R6, R7, R8, R9: footprint (none) -> Resistor_SMD:R_0402_1005Metric
- R12: value 100k -> 10k; footprint (none) -> Resistor_SMD:R_0402_1005Metric
- RV1, RV2: footprint (none) -> BreadModular_Pots:Potentiometer_RV09
- U1, U2: footprint (none) -> Package_SO:SOIC-8-1EP_3.9x4.9mm_P1.27mm_EP2.29x3mm
Connections:
- net +5V: now also C10.1, C11.1
- net GND: now also C10.2, C11.2
