File: modules/wave/wave.kicad_pcb (KiCad board)
At the start: 2 copper layers, 30.5 x 68.6 mm, 4 parts

Commit message: Initiate the PCB layut
Parts:
- added C1: 1nf, Capacitor_SMD:C_0402_1005Metric, F.Cu at (50.2, 44.5)
- added C10: 0.1uf, Capacitor_SMD:C_0402_1005Metric, F.Cu at (57.3, 85.7)
- added C11: 0.1uf, Capacitor_SMD:C_0402_1005Metric, F.Cu at (75.1, 85.5)
- added C2: 0.1uf, Capacitor_SMD:C_0402_1005Metric, F.Cu at (64.8, 86.9)
- added C3: 0.1uf, Capacitor_SMD:C_0402_1005Metric, F.Cu at (64.1, 89.4)
- added C4: 10nf, Capacitor_SMD:C_0402_1005Metric, F.Cu at (50.8, 46.8)
- added C5: 10nf, Capacitor_SMD:C_0402_1005Metric, F.Cu at (53.3, 46.8)
- added C6: 10nf, Capacitor_SMD:C_0402_1005Metric, F.Cu at (55.9, 46.8)
- added C7: 1uf, Capacitor_SMD:C_0402_1005Metric, F.Cu at (50.8, 49.4)
- added C8: 1uf, Capacitor_SMD:C_0402_1005Metric, F.Cu at (53.3, 49.4)
- added C9: 22uf, Capacitor_SMD:C_0805_2012Metric, F.Cu at (51.1, 53.3)
- added INPUT2: Caps, Connector_PinSocket_2.54mm:PinSocket_1x05_P2.54mm_Vertical, F.Cu at (55.9, 59.7)
- added R1: 1k, Resistor_SMD:R_0402_1005Metric, F.Cu at (73.7, 95.2)
- added R10: 100k, Resistor_SMD:R_0402_1005Metric, F.Cu at (66.8, 92.5)
- added R11: 100k, Resistor_SMD:R_0402_1005Metric, F.Cu at (67.3, 86.8)
- added R12: 10k, Resistor_SMD:R_0402_1005Metric, F.Cu at (66.8, 89.9)
- added R13: 1k, Resistor_SMD:R_0402_1005Metric, F.Cu at (69.7, 85.6)
- added R2: 1k, Resistor_SMD:R_0402_1005Metric, F.Cu at (71.1, 95.2)
- added R3: 100k, Resistor_SMD:R_0402_1005Metric, F.Cu at (50.2, 89.4)
- added R4: 100k, Resistor_SMD:R_0402_1005Metric, F.Cu at (49.7, 87.0)
- added R5: 10k, Resistor_SMD:R_0402_1005Metric, F.Cu at (52.8, 93.3)
- added R6: 1k, Resistor_SMD:R_0402_1005Metric, F.Cu at (49.7, 92.7)
- added R7: 100k, Resistor_SMD:R_0402_1005Metric, F.Cu at (60.2, 89.4)
- added R8: 100k, Resistor_SMD:R_0402_1005Metric, F.Cu at (59.7, 87.0)
- added R9: 1k, Resistor_SMD:R_0402_1005Metric, F.Cu at (59.7, 92.7)
- added RV1: 50k, BreadModular_Pots:Potentiometer_RV09, F.Cu at (52.1, 79.4)
- added RV2: 1M, BreadModular_Pots:Potentiometer_RV09, F.Cu at (67.3, 79.4)
- added U1: MCP6002-xSN, Package_SO:SOIC-8-1EP_3.9x4.9mm_P1.27mm_EP2.29x3mm, F.Cu at (72.3, 89.4)
- added U2: MCP6002-xSN, Package_SO:SOIC-8-1EP_3.9x4.9mm_P1.27mm_EP2.29x3mm, F.Cu at (54.7, 89.5)
- INPUT1: value Conn_01x05_Socket -> Cap Connect
- OUTPUT2: value Conn_01x05_Socket -> Output Waves
- moved INPUT1 12.5 mm to (55.9, 57.1), turned to 90 degrees
Connections:
- INPUT1 pad 1: unconnected-(INPUT1-Pin_1-Pad1) -> CAP_CONNECT
- INPUT1 pad 2: unconnected-(INPUT1-Pin_2-Pad2) -> CAP_CONNECT
- INPUT1 pad 3: unconnected-(INPUT1-Pin_3-Pad3) -> CAP_CONNECT
- INPUT1 pad 4: unconnected-(INPUT1-Pin_4-Pad4) -> CAP_CONNECT
- INPUT1 pad 5: unconnected-(INPUT1-Pin_5-Pad5) -> CAP_CONNECT
- OUTPUT2 pad 1: unconnected-(OUTPUT2-Pin_1-Pad1) -> OUT_SQUARE
- OUTPUT2 pad 2: unconnected-(OUTPUT2-Pin_2-Pad2) -> OUT_SQUARE
- OUTPUT2 pad 3: unconnected-(OUTPUT2-Pin_3-Pad3) -> OUT_TRI
- OUTPUT2 pad 4: unconnected-(OUTPUT2-Pin_4-Pad4) -> OUT_TRI
- OUTPUT2 pad 5: unconnected-(OUTPUT2-Pin_5-Pad5) -> OUT_SINE
Other:
- board text added: "C1"
- board text added: "C2"
- board text added: "CONFIG"
- board text added: "FINE"
- board text added: "FREQ"
- board text added: "HIGH"
- board text added: "LFO"
- board text added: "LOW"
- board text added: "WAVE"
- board text added: "WAVE 0.1.0"
- board text removed: "NAME"
- board text removed: "NAME 0.0.0"

Commit message: Finished PCB design.
Parts:
- moved C11 7.85 mm to (75.1, 93.3), turned to 180 degrees
- moved R8 2.54 mm to (59.8, 89.5), turned to 180 degrees
- moved R7 1.91 mm to (60.3, 87.5)
- moved R5 1.91 mm to (54.7, 93.3)
- moved R1 0.81 mm to (74.2, 95.9)
- moved C9 0.64 mm to (51.1, 52.7), turned to 180 degrees
- moved R2 0.64 mm to (71.1, 95.9)
- moved R9 0.12 mm to (59.7, 92.6), turned to -90 degrees
Routing:
- net GND: track 10.2 -> 135.0 mm, vias 0 -> 4
- net +5V: track 10.2 -> 111.9 mm, vias 0 -> 2
- net CAP_CONNECT: track 0.00 -> 89.3 mm, vias 0 -> 4
- net OUT_SQUARE: track 0.00 -> 72.5 mm, vias 0 -> 2
- net +2.5V: track 0.00 -> 70.4 mm, vias 0 -> 3
- net OUT_TRI: track 0.00 -> 52.9 mm, vias 0 -> 2
- net OPAMP_SQUARE: track 0.00 -> 48.7 mm
- net OUT_SINE: track 0.00 -> 34.3 mm
- net Net-(R5-Pad2): track 0.00 -> 30.9 mm, vias 0 -> 2
- net CAP_HIGH: track 0.00 -> 26.0 mm
- net CAP_CUSTOM: track 0.00 -> 23.3 mm, vias 0 -> 2
- net CAP_LOW: track 0.00 -> 20.9 mm
- net Net-(RV1-Pad3): track 0.00 -> 15.4 mm
- net CAP_LFO: track 0.00 -> 14.1 mm
- net Net-(C2-Pad2): track 0.00 -> 13.0 mm
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
Commit message: Add output wave captions.
Other:
- board text added: "OUTPUT"
- board text added: "SIN"
- board text added: "SQR"
- board text added: "TRI"
Changed lines of the file:
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@@
 		(property "Reference" "OUTPUT2"
 			(at -1.905 -2.54 0)
-			(layer "F.SilkS")
+			(layer "F.Fab")
 			(effects
 				(font
@@
 		)
 	)
+	(gr_poly
+		(pts
+			(xy 53.975 94.615) (xy 67.945 94.615) (xy 67.945 98.425) (xy 53.975 98.425)
+		)
+		(stroke
+			(width 0.2)
+			(type solid)
+		)
+		(fill solid)
+		(layer "B.Cu")
+		(net 1)
+	)
 	(gr_line
 		(start 46.99 109.22)
@@
 		(layer "Edge.Cuts")
 	)
+	(gr_text "SQR"
+		(at 71.501 46.355 0)
+		(layer "F.SilkS")
+		(effects
+			(font
+				(size 1 1)
+				(thickness 0.15)
+			)
+			(justify right bottom)
+		)
+	)
 	(gr_text "HIGH"
 		(at 61.595 61.57 90)
@@
 		)
 	)
+	(gr_text "SQR"
+		(at 71.501 48.895 0)
+		(layer "F.SilkS")
+		(effects
+			(font
+				(size 1 1)
+				(thickness 0.15)
+			)
+			(justify right bottom)
+		)
+	)
 	(gr_text "C1"
 		(at 64.135 61.57 90)
@@
 		)
 	)
+	(gr_text "TRI"
+		(at 71.501 53.975 0)
+		(layer "F.SilkS")
+		(effects
+			(font
+				(size 1 1)
+				(thickness 0.15)
+			)
+			(justify right bottom)
+		)
+	)
 	(gr_text "WAVE\n0.1.0"
 		(at 76.327 107.95 0)
@@
 		)
 	)
+	(gr_text "TRI"
+		(at 71.501 51.435 0)
+		(layer "F.SilkS")
+		(effects
+			(font
+				(size 1 1)
+				(thickness 0.15)
+			)
+			(justify right bottom)
+		)
+	)
 	(gr_text "C2"
 		(at 66.675 61.57 90)
@@
 		)
 	)
+	(gr_text "OUTPUT"
+		(at 75.057 43.942 0)
+		(layer "F.SilkS")
+		(effects
+			(font
+				(size 1 1)
+				(thickness 0.15)
+			)
+			(justify right bottom)
+		)
+	)
 	(gr_text "FINE"
 		(at 69.85 82.55 0)
@@
 		)
 	)
+	(gr_text "SIN"
+		(at 71.501 56.515 0)
+		(layer "F.SilkS")
+		(effects
+			(font
+				(size 1 1)
+				(thickness 0.15)
+			)
+			(justify right bottom)
+		)
+	)
