File: modules/usb_power/usb_power.kicad_sch (KiCad schematic)
At the start: 11 parts, among them J1 USB_C_Receptacle_PowerOnly_6P

Commit message: Changed the orientation of the USB C port
Parts:
- J1: footprint Connector_USB:USB_C_Receptacle_HRO_TYPE-C-31-M-12 -> BreadModular_TypeC:HRO-TYPE-C-31-M-12
Changed lines of the file:
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@@
 			)
 		)
-		(property "Footprint" "Connector_USB:USB_C_Receptacle_HRO_TYPE-C-31-M-12"
+		(property "Footprint" "BreadModular_TypeC:HRO-TYPE-C-31-M-12"
 			(at 73.66 52.07 0)
 			(effects
