File: modules/v2ca/v2ca.kicad_pcb (KiCad board)
At the start: 2 copper layers, 30.5 x 68.6 mm, 4 parts

Commit message: Finished the PCB layout.
Parts:
- removed OUTPUT2: Conn_01x05_Socket, Connector_PinSocket_2.54mm:PinSocket_1x05_P2.54mm_Vertical
- added C1: 0.1uf, Capacitor_SMD:C_0402_1005Metric, F.Cu at (69.1, 94.8)
- added C2: 0.1uf, Capacitor_SMD:C_0402_1005Metric, F.Cu at (66.2, 60.3)
- added C3: 0.1uf, Capacitor_SMD:C_0402_1005Metric, F.Cu at (58.6, 60.3)
- added OUTPUT1: Conn_01x05_Socket, Connector_PinSocket_2.54mm:PinSocket_1x05_P2.54mm_Vertical, F.Cu at (73.7, 45.7)
- added R1: 330, Resistor_SMD:R_0805_2012Metric, F.Cu at (52.3, 75.6)
- added R10: 10k, Resistor_SMD:R_0402_1005Metric, F.Cu at (72.5, 90.4)
- added R2: 1k, Resistor_SMD:R_0402_1005Metric, F.Cu at (70.2, 101.6)
- added R3: 10k, Resistor_SMD:R_0402_1005Metric, F.Cu at (74.9, 101.6)
- added R4: 10k, Resistor_SMD:R_0402_1005Metric, F.Cu at (72.5, 101.6)
- added R5: 1k, Resistor_SMD:R_0402_1005Metric, F.Cu at (63.4, 99.9)
- added R6: 1k, Resistor_SMD:R_0402_1005Metric, F.Cu at (60.3, 99.9)
- added R7: 330, Resistor_SMD:R_0805_2012Metric, F.Cu at (72.1, 75.6)
- added R8: 1k, Resistor_SMD:R_0402_1005Metric, F.Cu at (70.2, 90.4)
- added R9: 10k, Resistor_SMD:R_0402_1005Metric, F.Cu at (74.9, 90.4)
- added RV1: 50k, BreadModular_Pots:Potentiometer_RV09, F.Cu at (59.7, 73.7)
- added RV2: 50k, BreadModular_Pots:Potentiometer_RV09, F.Cu at (59.7, 90.6)
- added U1: VTL5C, BreadModular_MISC:VTL5C, B.Cu at (52.7, 75.6)
- added U2: MCP6002-xSN, Package_SO:SOIC-8-1EP_3.9x4.9mm_P1.27mm_EP2.29x3mm, F.Cu at (72.5, 96.3)
- added U3: VTL5C, BreadModular_MISC:VTL5C, B.Cu at (71.8, 75.6)
- added U4: MCP6002-xSN, Package_SO:SOIC-8-1EP_3.9x4.9mm_P1.27mm_EP2.29x3mm, F.Cu at (66.6, 57.1)
- added U5: MCP6002-xSN, Package_SO:SOIC-8-1EP_3.9x4.9mm_P1.27mm_EP2.29x3mm, F.Cu at (57.7, 57.1)
Connections:
- INPUT1 pad 1: unconnected-(INPUT1-Pin_1-Pad1) -> V1_IN
- INPUT1 pad 2: unconnected-(INPUT1-Pin_2-Pad2) -> CV1_IN
- INPUT1 pad 3: unconnected-(INPUT1-Pin_3-Pad3) -> V2_IN
- INPUT1 pad 4: unconnected-(INPUT1-Pin_4-Pad4) -> CV2_IN
Other:
- board text added: "CURVE 1"
- board text added: "CURVE 2"
- board text added: "CV1"
- board text added: "CV2"
- board text added: "IN1"
- board text added: "IN2"
- board text added: "INPUT"
- board text added: "MULT"
- board text added: "OUT1"
- board text added: "OUT2"
- board text added: "OUTPUT"

Commit message: Add the production version.
Parts:
- moved C3 6.41 mm to (52.4, 58.8), turned to 0 degrees
- moved R2 1.27 mm to (70.2, 102.9), turned to 180 degrees
- moved R3 1.27 mm to (74.9, 102.9)
- moved R4 1.27 mm to (72.5, 102.9)
- moved R5 1.02 mm to (63.4, 101.0)
- moved R6 1.02 mm to (60.3, 101.0)
- moved R10 0.89 mm to (71.6, 90.4)
- moved R9 0.89 mm to (74.0, 90.4)
- moved R8 0.89 mm to (69.3, 90.4)
Routing:
- net GND: track 10.2 -> 195.5 mm, vias 0 -> 5
- net +5V: track 10.2 -> 132.4 mm, vias 0 -> 6
- net V1_OUT: track 0.00 -> 63.1 mm, vias 0 -> 2
- net V2_OUT: track 0.00 -> 48.4 mm, vias 0 -> 2
- net Net-(R3-Pad1): track 0.00 -> 42.7 mm
- net Net-(U4B--): track 0.00 -> 39.8 mm, vias 0 -> 2
- net Net-(U5A--): track 0.00 -> 37.3 mm, vias 0 -> 2
- net Net-(U5B--): track 0.00 -> 31.0 mm, vias 0 -> 2
- net CV1_IN: track 0.00 -> 30.7 mm
- net CV2_IN: track 0.00 -> 29.6 mm, vias 0 -> 2
- net +2.5V: track 0.00 -> 28.2 mm, vias 0 -> 3
- net Net-(R7-Pad1): track 0.00 -> 27.0 mm
- net Net-(U4A--): track 0.00 -> 24.6 mm, vias 0 -> 2
- net V2_IN: track 0.00 -> 22.8 mm
- net V1_IN: track 0.00 -> 14.6 mm
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