File: modules/buff_mix/buff_mix.kicad_sch (KiCad schematic)
At the start: 2 parts

Commit message: Add the final buff_mix
Parts:
- added C1, C2, C3, C4, C5: C_Small, Capacitor_THT:C_Disc_D4.3mm_W1.9mm_P5.00mm, symbol Device:C_Small
- added INPUTS1, MIXOUT1: Conn_01x05_Socket, Connector_PinSocket_2.54mm:PinSocket_1x05_P2.54mm_Vertical, symbol Connector:Conn_01x05_Socket
- added R1, R2: 10K, Resistor_THT:R_Axial_DIN0207_L6.3mm_D2.5mm_P10.16mm_Horizontal, symbol Device:R
- added R3, R4, R5, R6, R7, R8: 100K, Resistor_THT:R_Axial_DIN0207_L6.3mm_D2.5mm_P10.16mm_Horizontal, symbol Device:R
- added U1, U2, U3: LM358, Library:LM358_THT, symbol Amplifier_Operational:LM358
Connections:
- net GND: now also R2.1, U1.4 (V-), U2.4 (V-), U3.4 (V-)
- net +5V: now reaches 5V1.1 (Pin_1)
- net +5V: now also 5V1.2 (Pin_2), 5V1.3 (Pin_3), 5V1.4 (Pin_4), 5V1.5 (Pin_5), R1.2, U1.8 (V+), U2.8 (V+), U3.8 (V+)
- new net: C3.2, R6.1
- new net: R3.1, R4.2, R5.2, R6.2, R7.2, R8.2, U1.6 (-)
- new net: C5.1, U3.6 (-), U3.7
- new net: C5.2, R8.1
- new net: C2.2, R5.1
- new net: C2.1, U2.1, U2.2 (-)
- new net: C1.2, R4.1
- new net: R1.1, R2.2, U1.5 (+)
- new net: C4.1, U3.1, U3.2 (-)
- new net: C4.2, R7.1
- new net: C3.1, U2.6 (-), U2.7
- new net: C1.1, U1.1, U1.2 (-)
- new net INPUT 1: INPUTS1.1 (Pin_1), U1.3 (+)
- new net INPUT 2: INPUTS1.2 (Pin_2), U2.3 (+)
- new net INPUT 3: INPUTS1.3 (Pin_3), U2.5 (+)
- new net INPUT 4: INPUTS1.4 (Pin_4), U3.3 (+)
- new net INPUT 5: INPUTS1.5 (Pin_5), U3.5 (+)
- new net MIX OUT: MIXOUT1.1 (Pin_1), MIXOUT1.2 (Pin_2), MIXOUT1.3 (Pin_3), MIXOUT1.4 (Pin_4), MIXOUT1.5 (Pin_5), R3.2, U1.7
Other:
- moved on the sheet: 5V1

Commit message: Designed the new buff_mix 0.2.0 schematic.
Parts:
- removed C1, C2, C3, C4, C5: C_Small, Capacitor_THT:C_Disc_D4.3mm_W1.9mm_P5.00mm, symbol Device:C_Small
- removed INPUTS1, MIXOUT1: Conn_01x05_Socket, Connector_PinSocket_2.54mm:PinSocket_1x05_P2.54mm_Vertical, symbol Connector:Conn_01x05_Socket
- removed U1, U2, U3: LM358, Library:LM358_THT, symbol Amplifier_Operational:LM358
- added C1, C2, C3, C4: 0.1uf, symbol Device:C
- added IN1, IN2, OUT1, OUT2: Conn_01x03_Socket, symbol Connector:Conn_01x03_Socket
- added R10, R13, R14, R15, R16, R18, R19, R20, R21, R22, R23, R24, R9: 1M, symbol Device:R
- added R11, R12, R17: 1k, symbol Device:R
- added RV1, RV2: 1M, symbol Device:R_Potentiometer
- added U1, U2, U3, U4: MCP6002-xSN, symbol Amplifier_Operational:MCP6002-xSN
- added V1: 5, symbol Simulation_SPICE:VDC
- added V2, V3, V4, V5, V6, V7: VSIN, symbol Simulation_SPICE:VSIN
- R1, R2: value 10K -> 1M; footprint Resistor_THT:R_Axial_DIN0207_L6.3mm_D2.5mm_P10.16mm_Horizontal -> (none)
- R3, R5, R6, R7, R8: value 100K -> 1M; footprint Resistor_THT:R_Axial_DIN0207_L6.3mm_D2.5mm_P10.16mm_Horizontal -> (none)
- R4: value 100K -> 1k; footprint Resistor_THT:R_Axial_DIN0207_L6.3mm_D2.5mm_P10.16mm_Horizontal -> (none)
Connections:
- net +5V: now also C1.1, C2.1, C3.1, C4.1, R11.1, U1.8 (V+), U2.8 (V+), U3.8 (V+), U4.8 (V+), V1.1; no longer R1.2
- net GND: now also C1.2, C2.2, C3.2, C4.2, R12.2, U1.4 (V-), U2.4 (V-), U3.4 (V-), U4.4 (V-), V1.2, V2.2, V3.2, V4.2, V5.2, V6.2, V7.2; no longer R2.1
- net at R6.1: now also RV1.3, U1.6 (-)
- net at R8.1: now also R7.2, U2.2 (-)
- net at R5.1: now also R8.2, U2.1
- net at R4.1: now also R6.2, U1.7
- net at R2.2: now also R3.1, U1.2 (-); no longer R1.1
- net INA_2: now reaches R7.1
- net INA_2: now also IN1.2 (Pin_2), V3.1
- net MIX OUT: no longer names the net of R3.2
- net MIX OUT: now also R1.1, U1.1
- new net: R23.2, R24.1, U4.6 (-)
- new net: R22.1, R24.2, U4.7
- new net: R15.2, R16.1, U3.2 (-)
- new net: R20.2, R21.1, U4.2 (-)
- new net: R14.1, R16.2, U3.1
- new net: R14.2, R18.2, R22.2, RV2.2
- new net: R19.1, RV2.3, U3.6 (-)
- new net: R17.1, R19.2, U3.7
- new net: R18.1, R21.2, U4.1
- new net: R10.2, R13.1, U2.6 (-)
- new net: R13.2, R9.1, U2.7
- new net: R1.2, R5.2, R9.2, RV1.2
- new net +2.5V: R11.2, R12.1, U1.3 (+), U1.5 (+), U2.3 (+), U2.5 (+), U3.3 (+), U3.5 (+), U4.3 (+), U4.5 (+)
- new net INA_1: IN1.1 (Pin_1), R2.1, V2.1
- new net INA_3: IN1.3 (Pin_3), R10.1, V4.1
- new net INB_1: IN2.1 (Pin_1), R15.1, V5.1
- new net INB_2: IN2.2 (Pin_2), R20.1, V6.1
- new net INB_3: IN2.3 (Pin_3), R23.1, V7.1
- new net OUTA: OUT1.1 (Pin_1), OUT1.2 (Pin_2), OUT1.3 (Pin_3), R4.2
- new net OUTB: OUT2.1 (Pin_1), OUT2.2 (Pin_2), OUT2.3 (Pin_3), R17.2
Other:
- moved on the sheet: 5V1, GND1

Commit message: Add the PCB layout of buff_mix
Parts:
- C1, C2, C3, C4: footprint (none) -> Capacitor_SMD:C_0402_1005Metric
- IN1, IN2, OUT1, OUT2: footprint (none) -> Connector_PinSocket_2.54mm:PinSocket_1x03_P2.54mm_Vertical
- R1, R10, R11, R12, R13, R14, R15, R16, R17, R18, R19, R2, R20, R21, R22, R23, R24, R3, R4, R5, R6, R7, R8, R9: footprint (none) -> Resistor_SMD:R_0402_1005Metric
- RV1, RV2: footprint (none) -> BreadModular_Pots:Potentiometer_RV09
- U1, U2, U3, U4: footprint (none) -> Package_SO:SOIC-8-1EP_3.9x4.9mm_P1.27mm_EP2.29x3mm
Changed lines of the file:
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@@
 			)
 		)
-		(property "Footprint" ""
+		(property "Footprint" "Resistor_SMD:R_0402_1005Metric"
 			(at 346.71 133.858 90)
 			(effects
@@
 			)
 		)
-		(property "Footprint" ""
+		(property "Footprint" "Resistor_SMD:R_0402_1005Metric"
 			(at 66.04 278.638 90)
 			(effects
@@
 			)
 		)
-		(property "Footprint" ""
+		(property "Footprint" "Resistor_SMD:R_0402_1005Metric"
 			(at 45.72 184.658 90)
 			(effects
@@
 			)
 		)
-		(property "Footprint" ""
+		(property "Footprint" "Resistor_SMD:R_0402_1005Metric"
 			(at 44.45 222.758 90)
 			(effects
@@
 			)
 		)
-		(property "Footprint" ""
+		(property "Footprint" "Resistor_SMD:R_0402_1005Metric"
 			(at 44.45 44.958 90)
 			(effects
@@
 			)
 		)
-		(property "Footprint" ""
+		(property "Footprint" "Resistor_SMD:R_0402_1005Metric"
 			(at 153.67 80.518 90)
 			(effects
@@
 			)
 		)
-		(property "Footprint" ""
+		(property "Footprint" "Connector_PinSocket_2.54mm:PinSocket_1x03_P2.54mm_Vertical"
 			(at 368.3 76.2 0)
 			(effects
@@
 			)
 		)
-		(property "Footprint" ""
+		(property "Footprint" "Resistor_SMD:R_0402_1005Metric"
 			(at 67.31 196.088 90)
 			(effects
@@
 			)
 		)
-		(property "Footprint" ""
+		(property "Footprint" "Resistor_SMD:R_0402_1005Metric"
 			(at 176.53 67.818 90)
 			(effects
@@
 			)
 		)
-		(property "Footprint" ""
+		(property "Footprint" "Connector_PinSocket_2.54mm:PinSocket_1x03_P2.54mm_Vertical"
 			(at 345.44 76.2 0)
 			(effects
@@
 			)
 		)
-		(property "Footprint" ""
+		(property "Footprint" "Package_SO:SOIC-8-1EP_3.9x4.9mm_P1.27mm_EP2.29x3mm"
 			(at 361.95 161.29 0)
 			(effects
@@
 			)
 		)
-		(property "Footprint" ""
+		(property "Footprint" "Resistor_SMD:R_0402_1005Metric"
 			(at 99.06 262.128 90)
 			(effects
@@
 			)
 		)
-		(property "Footprint" ""
+		(property "Footprint" "Package_SO:SOIC-8-1EP_3.9x4.9mm_P1.27mm_EP2.29x3mm"
 			(at 334.01 161.29 0)
 			(effects
@@
 			)
 		)
-		(property "Footprint" ""
+		(property "Footprint" "Connector_PinSocket_2.54mm:PinSocket_1x03_P2.54mm_Vertical"
 			(at 345.44 99.06 0)
 			(effects
@@
 			)
 		)
-		(property "Footprint" ""
+		(property "Footprint" "Package_SO:SOIC-8-1EP_3.9x4.9mm_P1.27mm_EP2.29x3mm"
 			(at 66.04 180.34 0)
 			(effects
@@
 			)
 		)
-		(property "Footprint" ""
+		(property "Footprint" "Package_SO:SOIC-8-1EP_3.9x4.9mm_P1.27mm_EP2.29x3mm"
 			(at 154.94 205.74 0)
 			(effects
@@
 			)
 		)
-		(property "Footprint" ""
+		(property "Footprint" "Resistor_SMD:R_0402_1005Metric"
 			(at 92.71 220.218 90)
 			(effects
@@
 			)
 		)
-		(property "Footprint" ""
+		(property "Footprint" "Capacitor_SMD:C_0402_1005Metric"
 			(at 338.7852 165.1 0)
 			(effects
@@
 			)
 		)
-		(property "Footprint" ""
+		(property "Footprint" "Package_SO:SOIC-8-1EP_3.9x4.9mm_P1.27mm_EP2.29x3mm"
 			(at 67.31 218.44 0)
 			(effects
@@
 			)
 		)
-		(property "Footprint" ""
+		(property "Footprint" "Resistor_SMD:R_0402_1005Metric"
 			(at 66.04 56.388 90)
 			(effects
@@
 			)
 		)
-		(property "Footprint" ""
+		(property "Footprint" "Resistor_SMD:R_0402_1005Metric"
 			(at 64.77 138.938 90)
 			(effects
@@
 			)
 		)
-		(property "Footprint" ""
+		(property "Footprint" "Resistor_SMD:R_0402_1005Metric"
 			(at 97.79 122.428 90)
 			(effects
@@
 			)
 		)
-		(property "Footprint" ""
+		(property "Footprint" "Package_SO:SOIC-8-1EP_3.9x4.9mm_P1.27mm_EP2.29x3mm"
 			(at 64.77 40.64 0)
 			(effects
@@
 			)
 		)
-		(property "Footprint" ""
+		(property "Footprint" "Capacitor_SMD:C_0402_1005Metric"
 			(at 366.7252 165.1 0)
 			(effects
@@
 			)
 		)
-		(property "Footprint" ""
+		(property "Footprint" "Resistor_SMD:R_0402_1005Metric"
 			(at 46.99 264.668 90)
 			(effects
@@
 			)
 		)
-		(property "Footprint" ""
+		(property "Footprint" "Connector_PinSocket_2.54mm:PinSocket_1x03_P2.54mm_Vertical"
 			(at 368.3 99.06 0)
 			(effects
@@
 			)
 		)
-		(property "Footprint" ""
+		(property "Footprint" "Capacitor_SMD:C_0402_1005Metric"
 			(at 395.9352 163.83 0)
 			(effects
@@
 			)
 		)
-		(property "Footprint" ""
+		(property "Footprint" "Package_SO:SOIC-8-1EP_3.9x4.9mm_P1.27mm_EP2.29x3mm"
 			(at 68.58 260.35 0)
 			(effects
@@
 			)
 		)
-		(property "Footprint" ""
+		(property "Footprint" "Package_SO:SOIC-8-1EP_3.9x4.9mm_P1.27mm_EP2.29x3mm"
 			(at 153.67 66.04 0)
 			(effects
@@
 			)
 		)
-		(property "Footprint" ""
+		(property "Footprint" "Resistor_SMD:R_0402_1005Metric"
 			(at 63.5 95.758 90)
 			(effects
@@
 			)
 		)
-		(property "Footprint" ""
+		(property "Footprint" "Package_SO:SOIC-8-1EP_3.9x4.9mm_P1.27mm_EP2.29x3mm"
 			(at 391.16 160.02 0)
 			(effects
@@
 			)
 		)
-		(property "Footprint" ""
+		(property "Footprint" "Resistor_SMD:R_0402_1005Metric"
 			(at 64.77 235.458 90)
 			(effects
@@
 			)
 		)
-		(property "Footprint" ""
+		(property "Footprint" "Resistor_SMD:R_0402_1005Metric"
 			(at 43.18 83.058 90)
 			(effects
@@
 			)
 		)
-		(property "Footprint" ""
+		(property "Footprint" "Resistor_SMD:R_0402_1005Metric"
 			(at 92.71 42.418 90)
 			(effects
@@
 			)
 		)
-		(property "Footprint" ""
+		(property "Footprint" "Resistor_SMD:R_0402_1005Metric"
 			(at 177.8 207.518 90)
 			(effects
@@
 			)
 		)
-		(property "Footprint" ""
+		(property "Footprint" "BreadModular_Pots:Potentiometer_RV09"
 			(at 127 68.58 0)
 			(effects
@@
 			)
 		)
-		(property "Footprint" ""
+		(property "Footprint" "Resistor_SMD:R_0402_1005Metric"
 			(at 361.95 133.858 90)
 			(effects
@@
 			)
 		)
-		(property "Footprint" ""
+		(property "Footprint" "Resistor_SMD:R_0402_1005Metric"
 			(at 45.72 124.968 90)
 			(effects
@@
 			)
 		)
-		(property "Footprint" ""
+		(property "Footprint" "Package_SO:SOIC-8-1EP_3.9x4.9mm_P1.27mm_EP2.29x3mm"
 			(at 66.04 78.74 0)
 			(effects
@@
 			)
 		)
-		(property "Footprint" ""
+		(property "Footprint" "Package_SO:SOIC-8-1EP_3.9x4.9mm_P1.27mm_EP2.29x3mm"
 			(at 304.8 162.56 0)
 			(effects
@@
 			)
 		)
-		(property "Footprint" ""
+		(property "Footprint" "BreadModular_Pots:Potentiometer_RV09"
 			(at 128.27 208.28 0)
 			(effects
@@
 			)
 		)
-		(property "Footprint" ""
+		(property "Footprint" "Resistor_SMD:R_0402_1005Metric"
 			(at 154.94 220.218 90)
 			(effects
@@
 			)
 		)
-		(property "Footprint" ""
+		(property "Footprint" "Package_SO:SOIC-8-1EP_3.9x4.9mm_P1.27mm_EP2.29x3mm"
 			(at 67.31 120.65 0)
 			(effects
@@
 			)
 		)
-		(property "Footprint" ""
+		(property "Footprint" "Resistor_SMD:R_0402_1005Metric"
 			(at 93.98 182.118 90)
 			(effects
@@
 			)
 		)
-		(property "Footprint" ""
+		(property "Footprint" "Resistor_SMD:R_0402_1005Metric"
 			(at 91.44 80.518 90)
 			(effects
@@
 			)
 		)
-		(property "Footprint" ""
+		(property "Footprint" "Capacitor_SMD:C_0402_1005Metric"
 			(at 309.5752 166.37 0)
 			(effects
