File: modules/line_in/line_in.kicad_pcb (KiCad board)
At the start: 2 copper layers, 30.5 x 68.6 mm, 28 parts, among them J1 AudioJack3, U1 MCP6002-xSN, U2 MCP6002-xSN, U3 MCP6002-xSN

Commit message: Add production line_in 0.2.0
Parts:
- R14: value 50k -> 51k
- R2, R8: value 24k -> 22k
Changed lines of the file:
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@@
 			)
 		)
-		(property "Value" "24k"
+		(property "Value" "22k"
 			(at 0 1.17 90)
 			(layer "F.Fab")
@@
 			)
 		)
-		(property "Value" "24k"
+		(property "Value" "22k"
 			(at 0 1.17 90)
 			(layer "F.Fab")
@@
 			)
 		)
-		(property "Value" "50k"
+		(property "Value" "51k"
 			(at 0 1.17 90)
 			(layer "F.Fab")
@@
 			)
 		)
+		(property "LCSC" "C7377"
+			(at 0 0 0)
+			(layer "F.SilkS")
+			(hide yes)
+			(effects
+				(font
+					(size 1.27 1.27)
+					(thickness 0.15)
+				)
+			)
+		)
 		(property ki_fp_filters "SOIC*3.9x4.9mm*P1.27mm* DIP*W7.62mm* TO*99* OnSemi*Micro8* TSSOP*3x3mm*P0.65mm* TSSOP*4.4x3mm*P0.65mm* MSOP*3x3mm*P0.65mm* SSOP*3.9x4.9mm*P0.635mm* LFCSP*2x2mm*P0.5mm* *SIP* SOIC*5.3x6.2mm*P1.27mm*")
 		(sheetname "Root")
@@
 			)
 		)
+		(property "LCSC" "C7377"
+			(at 0 0 0)
+			(layer "F.SilkS")
+			(hide yes)
+			(effects
+				(font
+					(size 1.27 1.27)
+					(thickness 0.15)
+				)
+			)
+		)
 		(property ki_fp_filters "SOIC*3.9x4.9mm*P1.27mm* DIP*W7.62mm* TO*99* OnSemi*Micro8* TSSOP*3x3mm*P0.65mm* TSSOP*4.4x3mm*P0.65mm* MSOP*3x3mm*P0.65mm* SSOP*3.9x4.9mm*P0.635mm* LFCSP*2x2mm*P0.5mm* *SIP* SOIC*5.3x6.2mm*P1.27mm*")
 		(sheetname "Root")
@@
 					(thickness 0.15)
 				)
+			)
+		)
+		(property "LCSC" "C7377"
+			(at 0 0 0)
+			(layer "F.SilkS")
+			(hide yes)
+			(effects
+				(font
+					(size 1.27 1.27)
+					(thickness 0.15)
+				)
