File: modules/line_in/line_in.kicad_sch (KiCad schematic)
At the start: 31 parts, among them J1 AudioJack3, U1 MCP6002-xSN, U2 MCP6002-xSN, U3 MCP6002-xSN

Commit message: Add production line_in 0.2.0
Parts:
- R14: value 50k -> 51k
- R2, R8: value 24k -> 22k
Changed lines of the file:
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@@
 			)
 		)
-		(property "Value" "50k"
+		(property "Value" "51k"
 			(at 92.71 165.1 90)
 			(effects
@@
 			)
 		)
-		(property "Value" "24k"
+		(property "Value" "22k"
 			(at 115.57 106.68 90)
 			(effects
@@
 			)
 		)
-		(property "Value" "24k"
+		(property "Value" "22k"
 			(at 115.57 63.5 90)
 			(effects
