File: modules/midi/esp32.kicad_sch (KiCad schematic)
At the start: 11 parts, among them J1 USB_C_Receptacle_USB2.0_16P, SW1 RESET, SW2 BOOT, U1 ESP32-S3-MINI-1U

Commit message: Add MIDI PCB
Parts:
- renumbered J1 to J4
Changed lines of the file:
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@@
 		(dnp no)
 		(fields_autoplaced yes)
-		(property "Reference" "#PWR014"
+		(property "Reference" "#PWR013"
 			(at 36.83 45.72 0)
 			(effects
@@
 			(project "midi"
 				(path "/b63493d3-5f6d-47e3-845b-87e7090fc1ab/49bb6b21-7f61-4812-af1a-818e74c87a72"
-					(reference "#PWR014")
+					(reference "#PWR013")
 					(unit 1)
 				)
@@
 		(dnp no)
 		(fields_autoplaced yes)
-		(property "Reference" "#PWR013"
+		(property "Reference" "#PWR016"
 			(at 53.34 49.53 0)
 			(effects
@@
 			(project "midi"
 				(path "/b63493d3-5f6d-47e3-845b-87e7090fc1ab/49bb6b21-7f61-4812-af1a-818e74c87a72"
-					(reference "#PWR013")
+					(reference "#PWR016")
 					(unit 1)
 				)
@@
 		(dnp no)
 		(fields_autoplaced yes)
-		(property "Reference" "#PWR012"
+		(property "Reference" "#PWR011"
 			(at 66.04 27.94 0)
 			(effects
@@
 			(project "midi"
 				(path "/b63493d3-5f6d-47e3-845b-87e7090fc1ab/49bb6b21-7f61-4812-af1a-818e74c87a72"
-					(reference "#PWR012")
+					(reference "#PWR011")
 					(unit 1)
 				)
@@
 		(dnp no)
 		(fields_autoplaced yes)
-		(property "Reference" "#PWR015"
+		(property "Reference" "#PWR017"
 			(at 66.04 57.15 0)
 			(effects
@@
 			(project "midi"
 				(path "/b63493d3-5f6d-47e3-845b-87e7090fc1ab/49bb6b21-7f61-4812-af1a-818e74c87a72"
-					(reference "#PWR015")
+					(reference "#PWR017")
 					(unit 1)
 				)
@@
 		(dnp no)
 		(fields_autoplaced yes)
-		(property "Reference" "#PWR018"
+		(property "Reference" "#PWR020"
 			(at 175.26 118.11 0)
 			(effects
@@
 			(project "midi"
 				(path "/b63493d3-5f6d-47e3-845b-87e7090fc1ab/49bb6b21-7f61-4812-af1a-818e74c87a72"
-					(reference "#PWR018")
+					(reference "#PWR020")
 					(unit 1)
 				)
@@
 		(dnp no)
 		(fields_autoplaced yes)
-		(property "Reference" "#PWR09"
+		(property "Reference" "#PWR012"
 			(at 113.03 27.94 0)
 			(effects
@@
 			(project "midi"
 				(path "/b63493d3-5f6d-47e3-845b-87e7090fc1ab/49bb6b21-7f61-4812-af1a-818e74c87a72"
-					(reference "#PWR09")
+					(reference "#PWR012")
 					(unit 1)
 				)
@@
 		(dnp no)
 		(fields_autoplaced yes)
-		(property "Reference" "#PWR08"
+		(property "Reference" "#PWR021"
 			(at 113.03 120.65 0)
 			(effects
@@
 			(project ""
 				(path "/b63493d3-5f6d-47e3-845b-87e7090fc1ab/49bb6b21-7f61-4812-af1a-818e74c87a72"
-					(reference "#PWR08")
+					(reference "#PWR021")
 					(unit 1)
 				)
@@
 		(dnp no)
 		(fields_autoplaced yes)
-		(property "Reference" "#PWR016"
+		(property "Reference" "#PWR018"
 			(at 36.83 74.93 0)
 			(effects
@@
 			(project "midi"
 				(path "/b63493d3-5f6d-47e3-845b-87e7090fc1ab/49bb6b21-7f61-4812-af1a-818e74c87a72"
-					(reference "#PWR016")
+					(reference "#PWR018")
 					(unit 1)
 				)
@@
 		(dnp no)
 		(fields_autoplaced yes)
-		(property "Reference" "#PWR011"
+		(property "Reference" "#PWR015"
 			(at 144.78 46.99 0)
 			(effects
@@
 			(project "midi"
 				(path "/b63493d3-5f6d-47e3-845b-87e7090fc1ab/49bb6b21-7f61-4812-af1a-818e74c87a72"
-					(reference "#PWR011")
+					(reference "#PWR015")
 					(unit 1)
 				)
@@
 		(dnp no)
 		(fields_autoplaced yes)
-		(property "Reference" "#PWR010"
+		(property "Reference" "#PWR014"
 			(at 124.46 46.99 0)
 			(effects
@@
 			(project "midi"
 				(path "/b63493d3-5f6d-47e3-845b-87e7090fc1ab/49bb6b21-7f61-4812-af1a-818e74c87a72"
-					(reference "#PWR010")
+					(reference "#PWR014")
 					(unit 1)
 				)
@@
 		(dnp no)
 		(fields_autoplaced yes)
-		(property "Reference" "#PWR017"
+		(property "Reference" "#PWR019"
 			(at 53.34 78.74 0)
 			(effects
@@
 			(project "midi"
 				(path "/b63493d3-5f6d-47e3-845b-87e7090fc1ab/49bb6b21-7f61-4812-af1a-818e74c87a72"
-					(reference "#PWR017")
+					(reference "#PWR019")
 					(unit 1)
 				)
@@
 		(dnp no)
 		(fields_autoplaced yes)
-		(property "Reference" "J1"
+		(property "Reference" "J4"
 			(at 175.26 55.88 0)
 			(effects
@@
 			(project ""
 				(path "/b63493d3-5f6d-47e3-845b-87e7090fc1ab/49bb6b21-7f61-4812-af1a-818e74c87a72"
-					(reference "J1")
-					(unit 1)
-				)
+					(reference "J4")
+					(unit 1)
+				)
