File: modules/midi/gate_process.kicad_sch (KiCad schematic)
At the start: 10 parts, among them U3 MCP6002-xSN

Commit message: Add MIDI PCB
Parts:
- renumbered C9 to C6, D3 to D1, R9 to R5, R8 to R7, R7 to R8

Commit message: Finalized the midi module.
Parts:
- removed unit 2 of U3
- removed unit 3 of U3
- added U2: MCP6002-xSN, Package_SO:SOIC-8-1EP_3.9x4.9mm_P1.27mm_EP2.29x3mm, symbol Amplifier_Operational:MCP6002-xSN
- renumbered U3 to U5
Connections:
- net GATE_B_IN: now also U2.5 (+)
- net GND: now also U2.4 (V-)
- net V_MID: now also U2.6 (-)
- net V_SUPPLY: now also U2.8 (V+)
- net at R8.1: now also U2.7
