File: modules/kick/kick.kicad_sch (KiCad schematic)
At the start: 33 parts, among them U1 MCP6002-xSN, U2 MCP6002-xSN, U3 VTL5C

Commit message: Assign footprints and PCB ready.
Parts:
- added C3: 100nf, Capacitor_SMD:C_0402_1005Metric, symbol Device:C
- added unit 3 of U1
- added unit 1 of U1
- added unit 2 of U3
- C1: renamed from C4; footprint (none) -> Capacitor_SMD:C_0402_1005Metric
- C2: renamed from C6; footprint (none) -> Capacitor_SMD:C_0402_1005Metric
- C4: renamed from C5; footprint (none) -> Capacitor_SMD:C_0402_1005Metric
- C5: renamed from C1; footprint (none) -> Capacitor_SMD:C_0402_1005Metric
- C6: renamed from C2; footprint (none) -> Capacitor_SMD:C_0402_1005Metric
- C7: renamed from C3; footprint (none) -> Capacitor_SMD:C_0402_1005Metric
- R1: renamed from R7; footprint (none) -> Resistor_SMD:R_0402_1005Metric
- R10: footprint (none) -> Resistor_SMD:R_0402_1005Metric
- R11: renamed from R8; footprint (none) -> Resistor_SMD:R_0402_1005Metric
- R12: renamed from R9; footprint (none) -> Resistor_SMD:R_0402_1005Metric
- R13: renamed from R11; footprint (none) -> Resistor_SMD:R_0402_1005Metric
- R14: renamed from R12; value 560 -> 10k; footprint (none) -> Resistor_SMD:R_0402_1005Metric
- R2: renamed from R1; footprint (none) -> Resistor_SMD:R_0402_1005Metric
- R3: renamed from R2; footprint (none) -> Resistor_SMD:R_0402_1005Metric
- R4: renamed from R5; footprint (none) -> Resistor_SMD:R_0402_1005Metric
- R5: renamed from R13; footprint (none) -> Resistor_SMD:R_0402_1005Metric
- R6: renamed from R14; footprint (none) -> Resistor_SMD:R_0402_1005Metric
- R7: renamed from R6; footprint (none) -> Resistor_SMD:R_0402_1005Metric
- R8: renamed from R3; footprint (none) -> Resistor_SMD:R_0402_1005Metric
- R9: renamed from R4; footprint (none) -> Resistor_SMD:R_0402_1005Metric
- RV1, RV2, RV3, RV4: footprint (none) -> BreadModular_Pots:Potentiometer_RV09
- U1, U2: footprint (none) -> Package_SO:SOIC-8-1EP_3.9x4.9mm_P1.27mm_EP2.29x3mm
- U2: renamed from U1; footprint (none) -> Package_SO:SOIC-8-1EP_3.9x4.9mm_P1.27mm_EP2.29x3mm
- U3: renamed from U2; footprint (none) -> Package_SO:SOIC-8-1EP_3.9x4.9mm_P1.27mm_EP2.29x3mm
- renumbered U3 to U4
Connections:
- net GATE_IN: now also INPUT1.1 (Pin_1), U1.3 (+); no longer C1.1
- net GND: now also C3.2, U1.4 (V-)
- net KICK_OUT: now also OUTPUT1.1 (Pin_1), OUTPUT1.2 (Pin_2), OUTPUT1.3 (Pin_3), OUTPUT1.4 (Pin_4), OUTPUT1.5 (Pin_5)
- net V_SUPPLY: now also C3.1, U1.8 (V+)
- net at INPUT1.2 (Pin_2): now also INPUT1.3 (Pin_3), INPUT1.4 (Pin_4), INPUT1.5 (Pin_5)
- new net: C1.1, U1.1, U1.2 (-)
Other:
- moved on the sheet: C1, C4, C5, R1, U2C, U3C

Commit message: Finished the 4 layer board.
Parts:
- U4: footprint OptoDevice:PerkinElmer_VTL5C -> BreadModular_MISC:VTL5C
Changed lines of the file:
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@@
 			)
 		)
-		(property "Footprint" "OptoDevice:PerkinElmer_VTL5C"
+		(property "Footprint" "BreadModular_MISC:VTL5C"
 			(at 52.07 208.28 0)
 			(effects

Commit message: Add production files.
Parts:
- added R15: 200k, Resistor_SMD:R_0402_1005Metric, symbol Device:R
- added R16: 51k, Resistor_SMD:R_0402_1005Metric, symbol Device:R
- R10: value 470k -> 200k
Connections:
- net CAP_MID: now also R16.2; no longer R10.2
- new net: R10.2, R15.1
- new net: R15.2, R16.1
Changed lines of the file:
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@@
 	(wire
 		(pts
+			(xy 236.22 172.72) (xy 237.49 172.72)
+		)
+		(stroke
+			(width 0)
+			(type default)
+		)
+	)
+	(wire
+		(pts
 			(xy 120.65 121.92) (xy 120.65 138.43)
 		)
@@
 	(wire
 		(pts
-			(xy 227.33 172.72) (xy 240.03 172.72)
+			(xy 227.33 172.72) (xy 228.6 172.72)
 		)
 		(stroke
@@
 	(wire
 		(pts
+			(xy 245.11 172.72) (xy 256.54 172.72)
+		)
+		(stroke
+			(width 0)
+			(type default)
+		)
+	)
+	(wire
+		(pts
 			(xy 106.68 138.43) (xy 110.49 138.43)
 		)
@@
 	(global_label "CAP_MID"
 		(shape bidirectional)
-		(at 240.03 172.72 0)
+		(at 256.54 172.72 0)
 		(fields_autoplaced yes)
 		(effects
@@
 		)
 		(property "Intersheetrefs" "${INTERSHEET_REFS}"
-			(at 252.0489 172.72 0)
+			(at 268.5589 172.72 0)
 			(effects
 				(font
@@
 	(symbol
 		(lib_id "Device:R")
+		(at 232.41 172.72 90)
+		(unit 1)
+		(exclude_from_sim no)
+		(in_bom yes)
+		(on_board yes)
+		(dnp no)
+		(fields_autoplaced yes)
+		(property "Reference" "R15"
+			(at 232.41 166.37 90)
+			(effects
+				(font
+					(size 1.27 1.27)
+				)
+			)
+		)
+		(property "Value" "200k"
+			(at 232.41 168.91 90)
+			(effects
+				(font
+					(size 1.27 1.27)
+				)
+			)
+		)
+		(property "Footprint" "Resistor_SMD:R_0402_1005Metric"
+			(at 232.41 174.498 90)
+			(effects
+				(font
+					(size 1.27 1.27)
+				)
+				(hide yes)
+			)
+		)
+		(property "Datasheet" "~"
+			(at 232.41 172.72 0)
+			(effects
+				(font
+					(size 1.27 1.27)
+				)
+				(hide yes)
+			)
+		)
+		(property "Description" "Resistor"
+			(at 232.41 172.72 0)
+			(effects
+				(font
+					(size 1.27 1.27)
+				)
+				(hide yes)
+			)
+		)
+		(pin "1"
+		)
+		(pin "2"
+		)
+		(instances
+			(project "kick"
+				(path "/b63493d3-5f6d-47e3-845b-87e7090fc1ab"
+					(reference "R15")
+					(unit 1)
+				)
+			)
+		)
+	)
+	(symbol
+		(lib_id "Device:R")
 		(at 144.78 115.57 180)
 		(unit 1)
@@
 			)
 		)
-		(property "Value" "470k"
+		(property "Value" "200k"
 			(at 223.52 168.91 90)
 			(effects
@@
 					(unit 1)
 				)
+			)
+		)
+	)
+	(symbol
+		(lib_id "Device:R")
+		(at 241.3 172.72 90)
+		(unit 1)
+		(exclude_from_sim no)
+		(in_bom yes)
+		(on_board yes)
+		(dnp no)
+		(fields_autoplaced yes)
+		(property "Reference" "R16"
+			(at 241.3 166.37 90)
+			(effects
+				(font
+					(size 1.27 1.27)
+				)
+			)
+		)
+		(property "Value" "51k"
+			(at 241.3 168.91 90)
+			(effects
+				(font
+					(size 1.27 1.27)
+				)
+			)
+		)
+		(property "Footprint" "Resistor_SMD:R_0402_1005Metric"
+			(at 241.3 174.498 90)
+			(effects
+				(font
+					(size 1.27 1.27)
+				)
+				(hide yes)
+			)
+		)
+		(property "Datasheet" "~"
+			(at 241.3 172.72 0)
+			(effects
+				(font
+					(size 1.27 1.27)
+				)
+				(hide yes)
+			)
+		)
+		(property "Description" "Resistor"
+			(at 241.3 172.72 0)
+			(effects
+				(font
+					(size 1.27 1.27)
+				)
+				(hide yes)
+			)
+		)
+		(pin "1"
+		)
+		(pin "2"
+		)
+		(instances
+			(project "kick"
+				(path "/b63493d3-5f6d-47e3-845b-87e7090fc1ab"
+					(reference "R16")
+					(unit 1)
+				)
