File: modules/drive/drive.kicad_sch (KiCad schematic)
At the start: 22 parts, among them U1 MCP6002-xSN

Commit message: drive: Remove radio freq. capturing with the gain. This is due to the high-gain nature & the use of non-inverting buffer. Now change it to an inverting buffer & all is gone.
Parts:
- added R7, R8: 100k, Resistor_SMD:R_0402_1005Metric, symbol Device:R
- RV2, RV3: value 1M -> 500k
Connections:
- net AUDIO_IN: now also R8.1; no longer U1.3 (+)
- net V_MID: now also U1.3 (+)
- net at RV1.2, U1.1: now also R7.2; no longer U1.2 (-)
- new net: R7.1, R8.2, U1.2 (-)
Changed lines of the file:
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@@
+	)
+	(junction
+		(at 49.53 76.2)
+		(diameter 0)
+		(color 0 0 0 0)
 	)
 	(junction
@@
 	(wire
 		(pts
+			(xy 46.99 76.2) (xy 49.53 76.2)
+		)
+		(stroke
+			(width 0)
+			(type default)
+		)
+	)
+	(wire
+		(pts
 			(xy 107.95 133.35) (xy 106.68 133.35)
 		)
@@
 	(wire
 		(pts
+			(xy 53.34 71.12) (xy 49.53 71.12)
+		)
+		(stroke
+			(width 0)
+			(type default)
+		)
+	)
+	(wire
+		(pts
+			(xy 64.77 87.63) (xy 72.39 87.63)
+		)
+		(stroke
+			(width 0)
+			(type default)
+		)
+	)
+	(wire
+		(pts
 			(xy 129.54 107.95) (xy 130.81 107.95)
 		)
@@
 	(wire
 		(pts
+			(xy 30.48 76.2) (xy 39.37 76.2)
+		)
+		(stroke
+			(width 0)
+			(type default)
+		)
+	)
+	(wire
+		(pts
 			(xy 111.76 88.9) (xy 106.68 88.9)
 		)
@@
 	(wire
 		(pts
-			(xy 41.91 71.12) (xy 53.34 71.12)
-		)
-		(stroke
-			(width 0)
-			(type default)
-		)
-	)
-	(wire
-		(pts
 			(xy 233.68 31.75) (xy 233.68 29.21)
 		)
@@
 	(wire
 		(pts
+			(xy 49.53 87.63) (xy 57.15 87.63)
+		)
+		(stroke
+			(width 0)
+			(type default)
+		)
+	)
+	(wire
+		(pts
 			(xy 135.89 62.23) (xy 135.89 74.93)
 		)
@@
 	(wire
 		(pts
-			(xy 72.39 83.82) (xy 49.53 83.82)
-		)
-		(stroke
-			(width 0)
-			(type default)
-		)
-	)
-	(wire
-		(pts
 			(xy 264.16 30.48) (xy 266.7 30.48)
 		)
@@
 	(wire
 		(pts
-			(xy 72.39 73.66) (xy 72.39 83.82)
+			(xy 72.39 73.66) (xy 72.39 87.63)
 		)
 		(stroke
@@
 	(wire
 		(pts
+			(xy 49.53 71.12) (xy 49.53 64.77)
+		)
+		(stroke
+			(width 0)
+			(type default)
+		)
+	)
+	(wire
+		(pts
 			(xy 106.68 77.47) (xy 107.95 77.47)
 		)
@@
 	(wire
 		(pts
-			(xy 49.53 83.82) (xy 49.53 76.2)
+			(xy 49.53 87.63) (xy 49.53 76.2)
 		)
 		(stroke
@@
 			(width 0)
 			(type default)
+		)
+	)
+	(global_label "V_MID"
+		(shape output)
+		(at 49.53 64.77 90)
+		(fields_autoplaced yes)
+		(effects
+			(font
+				(size 1.27 1.27)
+			)
+			(justify left)
+		)
+		(property "Intersheetrefs" "${INTERSHEET_REFS}"
+			(at 49.53 56.4024 90)
+			(effects
+				(font
+					(size 1.27 1.27)
+				)
+				(justify left)
+				(hide yes)
+			)
 		)
 	)
@@
 	(global_label "AUDIO_IN"
 		(shape input)
-		(at 41.91 71.12 180)
+		(at 30.48 76.2 180)
 		(fields_autoplaced yes)
 		(effects
@@
 		)
 		(property "Intersheetrefs" "${INTERSHEET_REFS}"
-			(at 30.3975 71.12 0)
+			(at 18.9675 76.2 0)
 			(effects
 				(font
@@
 			)
 		)
-		(property "Value" "1M"
+		(property "Value" "500k"
 			(at 125.73 114.3 90)
 			(effects
@@
 	(symbol
 		(lib_id "Device:R")
+		(at 60.96 87.63 90)
+		(unit 1)
+		(exclude_from_sim no)
+		(in_bom yes)
+		(on_board yes)
+		(dnp no)
+		(fields_autoplaced yes)
+		(property "Reference" "R7"
+			(at 60.96 81.28 90)
+			(effects
+				(font
+					(size 1.27 1.27)
+				)
+			)
+		)
+		(property "Value" "100k"
+			(at 60.96 83.82 90)
+			(effects
+				(font
+					(size 1.27 1.27)
+				)
+			)
+		)
+		(property "Footprint" "Resistor_SMD:R_0402_1005Metric"
+			(at 60.96 89.408 90)
+			(effects
+				(font
+					(size 1.27 1.27)
+				)
+				(hide yes)
+			)
+		)
+		(property "Datasheet" "~"
+			(at 60.96 87.63 0)
+			(effects
+				(font
+					(size 1.27 1.27)
+				)
+				(hide yes)
+			)
+		)
+		(property "Description" "Resistor"
+			(at 60.96 87.63 0)
+			(effects
+				(font
+					(size 1.27 1.27)
+				)
+				(hide yes)
+			)
+		)
+		(pin "1"
+		)
+		(pin "2"
+		)
+		(instances
+			(project "drive"
+				(path "/b63493d3-5f6d-47e3-845b-87e7090fc1ab"
+					(reference "R7")
+					(unit 1)
+				)
+			)
+		)
+	)
+	(symbol
+		(lib_id "Device:R")
 		(at 165.1 81.28 90)
 		(unit 1)
@@
 			)
 		)
-		(property "Value" "1M"
+		(property "Value" "500k"
 			(at 125.73 144.78 90)
 			(effects
@@
 					(unit 1)
 				)
+			)
+		)
+	)
+	(symbol
+		(lib_id "Device:R")
+		(at 43.18 76.2 90)
+		(unit 1)
+		(exclude_from_sim no)
+		(in_bom yes)
+		(on_board yes)
+		(dnp no)
+		(fields_autoplaced yes)
+		(property "Reference" "R8"
+			(at 43.18 69.85 90)
+			(effects
+				(font
+					(size 1.27 1.27)
+				)
+			)
+		)
+		(property "Value" "100k"
+			(at 43.18 72.39 90)
+			(effects
+				(font
+					(size 1.27 1.27)
+				)
+			)
+		)
+		(property "Footprint" "Resistor_SMD:R_0402_1005Metric"
+			(at 43.18 77.978 90)
+			(effects
+				(font
+					(size 1.27 1.27)
+				)
+				(hide yes)
+			)
+		)
+		(property "Datasheet" "~"
+			(at 43.18 76.2 0)
+			(effects
+				(font
+					(size 1.27 1.27)
+				)
+				(hide yes)
+			)
+		)
+		(property "Description" "Resistor"
+			(at 43.18 76.2 0)
+			(effects
+				(font
+					(size 1.27 1.27)
+				)
+				(hide yes)
+			)
+		)
+		(pin "1"
+		)
+		(pin "2"
+		)
+		(instances
+			(project "drive"
+				(path "/b63493d3-5f6d-47e3-845b-87e7090fc1ab"
+					(reference "R8")
+					(unit 1)
+				)
