File: modules/base/base.kicad_pcb (KiCad board)
At the start: 2 copper layers, 223.5 x 160 mm, 43 parts, among them J1 Power, J2 Ground, J3 Power, J4 Ground, J5 USB_C_Receptacle_PowerOnly_6P, U1 AMS1117-3.3

Commit message: base: Remove power extention via TRS cable Even with the regulator, it's noisy. So, instead now we use TRS only for syncing the ground between boards
Parts:
- J1, J3: value Power -> Ground
Connections:
- J1 pad T: +5V -> unconnected-(J1-PadT)
- J3 pad T: +5V -> unconnected-(J3-PadT)
Routing:
- net +5V: track 305.4 -> 17.7 mm
Other:
- board text added: "BASE 0.4.0"
- board text removed: "BASE 0.3.0"
- board text removed: "POWER (+5V)"
